Commit message: working on pick a cup

File: pickup_demo/mmp_panda.urdf (robot description, URDF)
Before this commit: robot mmp_panda, 13 links, 12 joints
Links:
- link link7: geometry collision mesh filename=../../../model/panda/meshes/collision/link7.obj; visual mesh filename=../../../model/panda/meshes/visual/hand.obj
- link rightfinger: geometry visual mesh filename=../../../model/panda/meshes/visual/finger.obj

Commit message: Robot aproaches object ready to grip

File: pickup_demo/mmp_panda.urdf (robot description, URDF)
Before this commit: robot mmp_panda, 13 links, 12 joints
Links:
- link link7: geometry collision mesh filename=../../../model/panda/meshes/collision/hand.obj; collision mesh filename=../../../model/panda/meshes/collision/link7.obj
