Commit message: basket fixed

File: grocery_robot/mmp_panda_no_basket.urdf (robot description, URDF)
Before this commit: robot mmp_panda, 18 links, 17 joints
Links:
- removed link basket_wall1
- removed link basket_wall2
- removed link basket_wall3
- removed link basket_wall4
- removed link basket_wall5
- link base_link: geometry visual mesh filename=../../../model/mmp_panda/meshes/panda_BaseCombo.obj
Joints:
- removed joint join_basket_0
- removed joint join_basket_1
- removed joint join_basket_2
- removed joint join_basket_3
- removed joint join_basket_4
