Commit message: final basket

File: grocery_robot/mmp_panda_basket.urdf (robot description, URDF)
Before this commit: robot mmp_panda, 13 links, 12 joints
Links:
- added link basket_wall1, mass 0.1; collision box size=0.005 0.5 0.25; visual box size=0.005 0.5 0.25
- added link basket_wall2, mass 0.1; collision box size=0.005 0.5 0.25; visual box size=0.005 0.5 0.25
- added link basket_wall3, mass 0.1; collision box size=0.29 0.005 0.24; visual box size=0.29 0.005 0.24
- added link basket_wall4, mass 0.1; collision box size=0.29 0.005 0.24; visual box size=0.29 0.005 0.24
- added link basket_wall5, mass 0.1; visual box size=0.3 0.5 0.005
Joints:
- added joint join_basket_0: type fixed, parent base_link, child basket_wall1, origin xyz=0.15 0.0 0.13 rpy=0 0 0, axis 0 0 1, limit lower=0 upper=6.28 effort=21.3 velocity=21.3
- added joint join_basket_1: type fixed, parent basket_wall1, child basket_wall2, origin xyz=0 0 0 rpy=0 0 0, axis 0 0 1, limit lower=0 upper=6.28 effort=21.3 velocity=21.3
- added joint join_basket_2: type fixed, parent basket_wall2, child basket_wall3, origin xyz=0 0 0 rpy=0 0 0, axis 0 0 1, limit lower=0 upper=6.28 effort=21.3 velocity=21.3
- added joint join_basket_3: type fixed, parent basket_wall3, child basket_wall4, origin xyz=0 0 0 rpy=0 0 0, axis 0 0 1, limit lower=0 upper=6.28 effort=21.3 velocity=21.3
- added joint join_basket_4: type fixed, parent basket_wall4, child basket_wall5, origin xyz=0 0 0 rpy=0 0 0, axis 0 0 1, limit lower=0 upper=6.28 effort=21.3 velocity=21.3

File: grocery_robot/mmp_panda_no_basket.urdf (robot description, URDF)
Before this commit: robot mmp_panda, 13 links, 12 joints
Links:
- link base_link: geometry collision box size=1 0.5 0.15; visual box size=0.6 0.5 0.15
