Commit message: basket created

File: grocery_robot/mmp_panda.urdf (robot description, URDF)
Before this commit: robot mmp_panda, 13 links, 12 joints
Links:
- added link basket_wall1, mass 0.1; collision box size=0.005 0.5 0.25; visual box size=0.005 0.5 0.25
- added link basket_wall2, mass 0.1; collision box size=0.005 0.5 0.25; visual box size=0.005 0.5 0.25
- added link basket_wall3, mass 0.1; collision box size=0.3 0.005 0.25; visual box size=0.3 0.005 0.25
- added link basket_wall4, mass 0.1; collision box size=0.3 0.005 0.25; visual box size=0.3 0.005 0.25
- added link basket_wall5, mass 0.1; collision box size=0.3 0.5 0.005; visual box size=0.3 0.5 0.005
Joints:
- added joint basket_link1: type fixed, parent base_link, child basket_wall1, origin xyz=0.25 0 0.15 rpy=0 0 0, axis 1 0 0
- added joint basket_link2: type fixed, parent basket_wall1, child basket_wall2, origin xyz=0 0 0 rpy=0 0 0, axis 0 1 0
- added joint basket_link3: type fixed, parent basket_wall2, child basket_wall3, origin xyz=0 0 0 rpy=0 0 0, axis 0 1 0
- added joint basket_link4: type fixed, parent basket_wall3, child basket_wall4, origin xyz=0 0 0 rpy=0 0 0, axis 0 1 0
- added joint basket_link5: type fixed, parent basket_wall4, child basket_wall5, origin xyz=0 0 0 rpy=0 0 0, axis 0 1 0

Commit message: pick working, errow basket waypoints

File: grocery_robot/mmp_panda.urdf (robot description, URDF)
Before this commit: robot mmp_panda, 18 links, 17 joints
Links:
- link base_link: geometry collision box size=1 0.5 0.15; visual box size=0.6 0.5 0.15

Commit message: leaving basket in conveyor

File: grocery_robot/mmp_panda.urdf (robot description, URDF)
Before this commit: robot mmp_panda, 13 links, 12 joints
Joints:
- joint base_prismatic_x: limit lower=-2.8973 upper=2.9873 effort=87 velocity=2.1750 -> lower=-5 upper=5 effort=87 velocity=2.1750
- joint base_prismatic_y: limit lower=-2.8973 upper=2.9873 effort=87 velocity=2.1750 -> lower=-5 upper=5 effort=87 velocity=2.1750
- joint base_revolute: limit lower=-2.8973 upper=2.8973 effort=87 velocity=2.1750 -> lower=-5 upper=5 effort=87 velocity=2.1750
